File: hardware/cmos-imx179/cmos-imx179-breakout.kicad_pcb (KiCad board)
At the start: 4 copper layers, 30 x 16.9 mm, 55 parts, among them J1 Conn_01x20, U1 NCP167, U2 NCP167, U3 imx179-plcc40, U4 NCP167, U5 24.00MHz

Commit message: Updated CMOS IMX179 Breakout
Parts:
- C1, C10, C11, C3, C5, C9: value 1u -> 1uF
- C12, C13, C14, C15, C16, C17, C18, C19, C20, C21, C22, C23, C24, C25, C7: value 100n -> 100nF
- G*** (x2): moved to B.Cu
- R1, R2: value 2K2 -> 2.2K
- U1: value NCP167 -> NCP114-120
- U2: value NCP167 -> NCP167-180
- U4: value NCP167 -> NCP167-270
- U5: value 24.00MHz -> 24.00 MHz
- moved G*** 11.8 mm to (138.1, 90.6), turned to 180 degrees
- moved G*** 11.0 mm to (138.1, 88.4), turned to 180 degrees
Connections:
- J1 pad 16: /FPGA_IO_0 -> /ENABLE
Routing:
- net /ENABLE: track 33.9 -> 43.0 mm
- net +1V2: track 34.4 -> 36.1 mm
Other:
- board text added: "2019-03-23"
